File: hw/sch_pcb/SATABAL01A.kicad_pcb (KiCad board)
At the start: 2 copper layers, 40.1 x 30 mm, 9 parts, among them J1 SATA7-67491-1030, J2 Conn_Coaxial SMA or MCX, J3 Conn_Coaxial SMA or MCX, T1 ETC1-1-13, T2 ETC1-1-13

Commit message: výrobní data
Other:
- rule pad_to_mask_clearance: 0 -> 0.2
Changed lines of the file:
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@@
       (dielectric_constraints no)
     )
-    (pad_to_mask_clearance 0)
+    (pad_to_mask_clearance 0.2)
     (pcbplotparams
       (layerselection 0x00010e0_ffffffff)
