File: hw/sch_pcb/SATABAL01A.kicad_sch (KiCad schematic)
At the start: 9 parts, among them J1 SATA7-67491-1030, J2 Conn_Coaxial SMA or MCX, J3 Conn_Coaxial SMA or MCX, T1 ETC1-1-13, T2 ETC1-1-13

Commit message: Add mathing UST_ID to components. #1
Parts:
- J1: UST_ID (none) -> 5c70984712875079b91f8a7b
- J2, J3: UST_ID (none) -> 5c70984412875079b91f87ac
- T1, T2: UST_ID (none) -> 5face38612875025b3977e95
Changed lines of the file:
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@@
+      (effects (font (size 1.27 1.27)) hide)
+    )
+    (property "UST_ID" "5c70984412875079b91f87ac" (id 4) (at 228.6 95.885 0)
       (effects (font (size 1.27 1.27)) hide)
     )
@@
       (effects (font (size 1.27 1.27)) hide)
     )
+    (property "UST_ID" "5c70984412875079b91f87ac" (id 4) (at 229.87 65.405 0)
+      (effects (font (size 1.27 1.27)) hide)
+    )
     (pin "1")
     (pin "2")
@@
     (property "Datasheet" "" (id 3) (at 59.69 88.9 0)
       (effects (font (size 1.524 1.524)))
+    )
+    (property "UST_ID" "5c70984712875079b91f8a7b" (id 4) (at 59.69 88.9 0)
+      (effects (font (size 1.27 1.27)) hide)
     )
     (pin "1")
@@
       (effects (font (size 1.27 1.27)) hide)
     )
+    (property "UST_ID" "5face38612875025b3977e95" (id 4) (at 149.86 67.31 0)
+      (effects (font (size 1.27 1.27)) hide)
+    )
     (pin "1")
     (pin "2")
@@
       (effects (font (size 1.27 1.27)) hide)
     )
+    (property "UST_ID" "5face38612875025b3977e95" (id 4) (at 149.86 96.52 0)
+      (effects (font (size 1.27 1.27)) hide)
+    )
